File: PCB/Skeleton8.kicad_pcb (KiCad board)
At the start: 2 copper layers, 97.6 x 95.2 mm, 70 parts, among them J1 TYPE-C-31-M-12, Q1 SI2302, SW1 SW_Push, SW2 SW_Push, SW3 SW_Push, SW4 SW_Push, SW5 SW_Push, SW6 SW_Push, SW7 SW_Push, SW8 SW_Push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

Commit message: v1
Parts:
- removed FID1, FID2, FID3, FID4: Fiducial, Fiducial:Fiducial_1mm_Mask2mm
- added H1: Hole, project:ToolingHole, F.Cu at (48.9, 51.0)
- added H2: Hole, project:ToolingHole, F.Cu at (51.8, 81.3)
- added H3: Hole, project:ToolingHole, F.Cu at (120.0, 84.4)
Routing:
- net Net-(Q1-D): track 161.8 -> 163.6 mm
- net +1V1: track 81.5 -> 82.4 mm
Other:
- board size 97.6 x 95.2 mm -> 81 x 52.4 mm
- board text added: "BOOT"
- board text added: "RESET"
- board text removed: "<- V-Cut"
