File: PCB/Skeleton8.kicad_sch (KiCad schematic)
At the start: 70 parts, among them J1 TYPE-C-31-M-12, Q1 SI2302, SW1 SW_Push, SW2 SW_Push, SW3 SW_Push, SW4 SW_Push, SW5 SW_Push, SW6 SW_Push, SW7 SW_Push, SW8 SW_Push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

Commit message: v1
Parts:
- removed FID1, FID2, FID3, FID4: Fiducial, Fiducial:Fiducial_1mm_Mask2mm, symbol Mechanical:Fiducial
- added H1, H2, H3: Hole, project:ToolingHole, symbol keebio:Hole
Changed lines of the file:
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@@
-    )
-  )
-  (symbol (lib_id "Mechanical:Fiducial") (at 18.415 184.15 0) (unit 1)
-    (in_bom yes) (on_board yes) (dnp no) (fields_autoplaced)
-    (property "Reference" "FID4" (at 20.955 182.8799 0)
-      (effects (font (size 1.27 1.27)) (justify left))
-    )
-    (property "Value" "Fiducial" (at 20.955 185.4199 0)
-      (effects (font (size 1.27 1.27)) (justify left))
-    )
-    (property "Footprint" "Fiducial:Fiducial_1mm_Mask2mm" (at 18.415 184.15 0)
-      (effects (font (size 1.27 1.27)) hide)
-    )
-    (property "Datasheet" "~" (at 18.415 184.15 0)
-      (effects (font (size 1.27 1.27)) hide)
-    )
-    (instances
-      (project "Skeleton8"
-        (path "/27f80fc5-9574-4484-9163-c7fd64f457f7"
-          (reference "FID4") (unit 1)
-        )
-      )
-      (project "Skeleton68rev2"
-        (path "/8e88366a-267f-41cf-9fb4-3c55e34173db"
-          (reference "FID4") (unit 1)
-        )
-      )
     )
   )
@@
         (path "/8e88366a-267f-41cf-9fb4-3c55e34173db"
           (reference "C12") (unit 1)
-        )
-      )
-    )
-  )
-  (symbol (lib_id "Mechanical:Fiducial") (at 18.415 180.34 0) (unit 1)
-    (in_bom yes) (on_board yes) (dnp no) (fields_autoplaced)
-    (property "Reference" "FID3" (at 20.955 179.0699 0)
-      (effects (font (size 1.27 1.27)) (justify left))
-    )
-    (property "Value" "Fiducial" (at 20.955 181.6099 0)
-      (effects (font (size 1.27 1.27)) (justify left))
-    )
-    (property "Footprint" "Fiducial:Fiducial_1mm_Mask2mm" (at 18.415 180.34 0)
-      (effects (font (size 1.27 1.27)) hide)
-    )
-    (property "Datasheet" "~" (at 18.415 180.34 0)
-      (effects (font (size 1.27 1.27)) hide)
-    )
-    (instances
-      (project "Skeleton8"
-        (path "/27f80fc5-9574-4484-9163-c7fd64f457f7"
-          (reference "FID3") (unit 1)
-        )
-      )
-      (project "Skeleton68rev2"
-        (path "/8e88366a-267f-41cf-9fb4-3c55e34173db"
-          (reference "FID3") (unit 1)
         )
       )
@@
     )
   )
-  (symbol (lib_id "Mechanical:Fiducial") (at 18.415 172.72 0) (unit 1)
-    (in_bom yes) (on_board yes) (dnp no) (fields_autoplaced)
-    (property "Reference" "FID1" (at 20.955 171.4499 0)
-      (effects (font (size 1.27 1.27)) (justify left))
-    )
-    (property "Value" "Fiducial" (at 20.955 173.9899 0)
-      (effects (font (size 1.27 1.27)) (justify left))
-    )
-    (property "Footprint" "Fiducial:Fiducial_1mm_Mask2mm" (at 18.415 172.72 0)
-      (effects (font (size 1.27 1.27)) hide)
-    )
-    (property "Datasheet" "~" (at 18.415 172.72 0)
-      (effects (font (size 1.27 1.27)) hide)
-    )
-    (instances
-      (project "Skeleton8"
-        (path "/27f80fc5-9574-4484-9163-c7fd64f457f7"
-          (reference "FID1") (unit 1)
-        )
-      )
-      (project "Skeleton68rev2"
-        (path "/8e88366a-267f-41cf-9fb4-3c55e34173db"
-          (reference "FID1") (unit 1)
-        )
-      )
-    )
-  )
   (symbol (lib_id "custom:WS2812B-2020") (at 410.21 180.34 0) (unit 1)
     (in_bom yes) (on_board yes) (dnp no)
@@
     )
   )
+  (symbol (lib_id "keebio:Hole") (at 266.7 24.13 0) (unit 1)
+    (in_bom yes) (on_board yes) (dnp no) (fields_autoplaced)
+    (property "Reference" "H3" (at 271.78 22.86 0)
+      (effects (font (size 1.524 1.524)) (justify left))
+    )
+    (property "Value" "Hole" (at 271.78 25.4 0)
+      (effects (font (size 1.524 1.524)) (justify left))
+    )
+    (property "Footprint" "project:ToolingHole" (at 266.7 24.13 0)
+      (effects (font (size 1.524 1.524)) hide)
+    )
+    (property "Datasheet" "" (at 266.7 24.13 0)
+      (effects (font (size 1.524 1.524)) hide)
+    )
+    (instances
+      (project "Skeleton8"
+        (path "/27f80fc5-9574-4484-9163-c7fd64f457f7"
+          (reference "H3") (unit 1)
+        )
+      )
+    )
+  )
   (symbol (lib_name "PWR_FLAG_1") (lib_id "power:PWR_FLAG") (at 77.47 25.4 0) (unit 1)
     (in_bom yes) (on_board yes) (dnp no) (fields_autoplaced)
@@
         (path "/27f80fc5-9574-4484-9163-c7fd64f457f7"
           (reference "#FLG03") (unit 1)
-        )
-      )
-    )
-  )
-  (symbol (lib_id "Mechanical:Fiducial") (at 18.415 176.53 0) (unit 1)
-    (in_bom yes) (on_board yes) (dnp no) (fields_autoplaced)
-    (property "Reference" "FID2" (at 20.955 175.2599 0)
-      (effects (font (size 1.27 1.27)) (justify left))
-    )
-    (property "Value" "Fiducial" (at 20.955 177.7999 0)
-      (effects (font (size 1.27 1.27)) (justify left))
-    )
-    (property "Footprint" "Fiducial:Fiducial_1mm_Mask2mm" (at 18.415 176.53 0)
-      (effects (font (size 1.27 1.27)) hide)
-    )
-    (property "Datasheet" "~" (at 18.415 176.53 0)
-      (effects (font (size 1.27 1.27)) hide)
-    )
-    (instances
-      (project "Skeleton8"
-        (path "/27f80fc5-9574-4484-9163-c7fd64f457f7"
-          (reference "FID2") (unit 1)
-        )
-      )
-      (project "Skeleton68rev2"
-        (path "/8e88366a-267f-41cf-9fb4-3c55e34173db"
-          (reference "FID2") (unit 1)
         )
       )
@@
         (path "/8e88366a-267f-41cf-9fb4-3c55e34173db"
           (reference "C10") (unit 1)
+        )
+      )
+    )
+  )
+  (symbol (lib_id "keebio:Hole") (at 248.92 24.13 0) (unit 1)
+    (in_bom yes) (on_board yes) (dnp no) (fields_autoplaced)
+    (property "Reference" "H2" (at 254 22.86 0)
+      (effects (font (size 1.524 1.524)) (justify left))
+    )
+    (property "Value" "Hole" (at 254 25.4 0)
+      (effects (font (size 1.524 1.524)) (justify left))
+    )
+    (property "Footprint" "project:ToolingHole" (at 248.92 24.13 0)
+      (effects (font (size 1.524 1.524)) hide)
+    )
+    (property "Datasheet" "" (at 248.92 24.13 0)
+      (effects (font (size 1.524 1.524)) hide)
+    )
+    (instances
+      (project "Skeleton8"
+        (path "/27f80fc5-9574-4484-9163-c7fd64f457f7"
+          (reference "H2") (unit 1)
         )
       )
@@
         )
       )
+    )
+  )
+  (symbol (lib_id "keebio:Hole") (at 231.14 24.13 0) (unit 1)
+    (in_bom yes) (on_board yes) (dnp no) (fields_autoplaced)
+    (property "Reference" "H1" (at 236.22 22.86 0)
+      (effects (font (size 1.524 1.524)) (justify left))
+    )
+    (property "Value" "Hole" (at 236.22 25.4 0)
+      (effects (font (size 1.524 1.524)) (justify left))
+    )
+    (property "Footprint" "project:ToolingHole" (at 231.14 24.13 0)
+      (effects (font (size 1.524 1.524)) hide)
+    )
+    (property "Datasheet" "" (at 231.14 24.13 0)
+      (effects (font (size 1.524 1.524)) hide)
+    )
+    (instances
+      (project "Skeleton8"
+        (path "/27f80fc5-9574-4484-9163-c7fd64f457f7"
+          (reference "H1") (unit 1)
+        )
+      )
